Commit message: feat(gripper): add gripper controllers, calibrate gz_ros2_control gains, and clean environment assets

File: src/franka_description/end_effectors/common/franka_hand.xacro (robot description, xacro)
@@ -117,5 +117,5 @@
       <origin xyz="0 0 0.0584" rpy="0 0 0" />
       <axis xyz="0 1 0" />
-      <limit effort="100" lower="0.0" upper="0.04" velocity="0.2" />
+      <limit effort="100" lower="-0.005" upper="0.05" velocity="0.2" />
       <dynamics damping="0.3" />
     </joint>
@@ -125,5 +125,5 @@
       <origin xyz="0 0 0.0584" rpy="0 0 ${pi}" />
       <axis xyz="0 1 0" />
-      <limit effort="100" lower="0.0" upper="0.04" velocity="0.2" />
+      <limit effort="100" lower="-0.005" upper="0.05" velocity="0.2" />
       <mimic joint="${ee_prefix}finger_joint1" />
       <dynamics damping="0.3" />

File: src/franka_ros2/franka_gazebo/franka_gazebo_bringup/urdf/environment_assets.xacro (robot description, xacro)
@@ -72,29 +72,3 @@
   <xacro:shelf_macro prefix="shelf_1" parent="world" x="0.0" y="-1.2" z="0.0"/>
   <xacro:shelf_macro prefix="shelf_2" parent="world" x="0.0" y="1.2" z="0.0"/>
-  <!-- ================= HEDEF KIRMIZI KUTU (TARGET BOX) ================= -->
-  <!-- 2. Kat tablası Z = 0.45m'de. Tabla kalınlığı 0.025m, kutu 0.05m -> Z_merkez = 0.45 + 0.0125 + 0.025 = 0.4875m -->
-  <link name="target_box_link">
-    <inertial>
-      <mass value="0.05"/>
-      <origin xyz="0 0 0" rpy="0 0 0"/>
-      <inertia ixx="0.00002" ixy="0" ixz="0" iyy="0.00002" iyz="0" izz="0.00002"/>
-    </inertial>
-    <visual>
-      <origin xyz="0 0 0" rpy="0 0 0"/>
-      <geometry><box size="0.05 0.05 0.05"/></geometry>
-      <material name="bright_red"><color rgba="1.0 0.0 0.0 1.0"/></material>
-    </visual>
-    <collision>
-      <origin xyz="0 0 0" rpy="0 0 0"/>
-      <geometry><box size="0.05 0.05 0.05"/></geometry>
-    </collision>
-  </link>
-  <joint name="target_box_joint" type="fixed">
-    <parent link="shelf_1_link"/>
-    <child link="target_box_link"/>
-    <origin xyz="0.0 0.0 0.4875" rpy="0 0 0"/>
-  </joint>
-  <gazebo reference="target_box_link">
-    <material>Gazebo/Red</material>
-  </gazebo>
 </robot>

File: src/franka_ros2/franka_gazebo/franka_gazebo_bringup/urdf/franka_gazebo_hardware_plugins.xacro (robot description, xacro)
@@ -28,4 +28,5 @@
       <plugin filename="gz_ros2_control-system" name="gz_ros2_control::GazeboSimROS2ControlPlugin">
         <parameters>$(find franka_gazebo_bringup)/config/franka_gazebo_controllers.yaml</parameters>
+        <position_proportional_gain>0.002</position_proportional_gain>
       </plugin>
     </gazebo>
